Commit message: work in progress

File: config/dome1_tf_only.urdf.xacro (robot description, xacro)
@@ -13,6 +13,6 @@
   <link name="base_link"/>
   <joint name="base_link_to_base_footprint" type="fixed">
-    <parent link="base_link"/>
-    <child link="base_footprint"/>
+    <parent link="base_footprint"/>
+    <child link="base_link"/>
     <origin xyz="${-base_link_x_offset} 0 ${-bottom_plate_height}" rpy="0 0 0"/>
   </joint>

Commit message: work in progress

File: config/dome1_tf_only.urdf.xacro (robot description, xacro)
@@ -8,11 +8,11 @@
   <xacro:property name="imu_x_offset" value="-0.040" />
   <xacro:property name="imu_z_offset" value="0.020" />
+  <!-- Base link (main robot body) -->
+  <link name="base_link"/>
   <!-- Base footprint (ground projection) -->
   <link name="base_footprint"/>
-  <!-- Base link (main robot body) -->
-  <link name="base_link"/>
   <joint name="base_link_to_base_footprint" type="fixed">
-    <parent link="base_footprint"/>
-    <child link="base_link"/>
+    <parent link="base_link"/>
+    <child link="base_footprint"/>
     <origin xyz="${-base_link_x_offset} 0 ${-bottom_plate_height}" rpy="0 0 0"/>
   </joint>
