Commit message: changed so that we get the official slam and nav2 yaml configs from the paclates and then patch them within dome

File: config/dome2.urdf (robot description, URDF)
Before this commit: robot dome2, 15 links, 14 joints
Links:
- removed link imu_back_link
- removed link imu_bottom_link
- removed link imu_front_link
- removed link imu_right_link
- removed link imu_top_link
- added link imu_forward_link; collision box size=0.03 0.002 0.002; visual box size=0.03 0.002 0.002
- added link imu_up_link; collision box size=0.002 0.002 0.03; visual box size=0.002 0.002 0.03
- added link laser_forward_link; collision box size=0.04 0.002 0.002; visual box size=0.04 0.002 0.002
- added link laser_left_link; collision box size=0.002 0.04 0.002; visual box size=0.002 0.04 0.002
- added link laser_up_link; collision box size=0.002 0.002 0.04; visual box size=0.002 0.002 0.04
- link imu_left_link: geometry collision box size=0.002 0.03 0.002; visual box size=0.002 0.03 0.002
- link imu_link: geometry collision box size=0.03 0.02 0.01; visual box size=0.03 0.02 0.01
Joints:
- removed joint imu_link_to_imu_back_link
- removed joint imu_link_to_imu_bottom_link
- removed joint imu_link_to_imu_front_link
- removed joint imu_link_to_imu_right_link
- removed joint imu_link_to_imu_top_link
- added joint imu_link_to_imu_forward_link: type fixed, parent imu_link, child imu_forward_link, origin xyz=0.015 0 0
- added joint imu_link_to_imu_up_link: type fixed, parent imu_link, child imu_up_link, origin xyz=0 0 0.015
- added joint laser_to_laser_forward_link: type fixed, parent laser, child laser_forward_link, origin xyz=0.02 0 0
- added joint laser_to_laser_left_link: type fixed, parent laser, child laser_left_link, origin xyz=0 0.02 0
- added joint laser_to_laser_up_link: type fixed, parent laser, child laser_up_link, origin xyz=0 0 0.03
- joint base_link_to_laser: origin xyz=0 0 0.1 -> xyz=0 0 0.1 rpy=0 0 -1.5707963267948966
- joint imu_link_to_imu_left_link: origin xyz=0 0.0095 0 -> xyz=0 0.01 0

Commit message: tuning dome2

File: config/dome2.urdf (robot description, URDF)
Before this commit: robot dome2, 15 links, 14 joints
Joints:
- joint base_link_to_imu_link: origin xyz=0.03 0 0.053 rpy=1.5707963267948966 0 3.141592653589793 -> xyz=0.05 0 0.01 rpy=0 0 0

Commit message: continued tuning

File: config/dome2.urdf (robot description, URDF)
Before this commit: robot dome2, 15 links, 14 joints
Joints:
- joint base_link_to_imu_link: origin xyz=0.05 0 0.01 rpy=0 0 0 -> xyz=0.0 0 0.05 rpy=0 0 0
- joint base_link_to_laser: origin xyz=0 0 0.1 rpy=0 0 -1.5707963267948966 -> xyz=-0.15 0 0.1 rpy=0 0 -1.5707963267948966
