Commit message: work in progress

File: install/dome/share/dome/config/dome1.urdf.xacro (robot description, xacro)
@@ -50,6 +50,6 @@
   <link name="base_link"/>
   <joint name="base_link_to_base_footprint" type="fixed">
-    <parent link="base_link"/>
-    <child link="base_footprint"/>
+    <parent link="base_footprint"/>
+    <child link="base_link"/>
     <origin xyz="${-base_link_x_offset} 0 ${-bottom_plate_height}" rpy="0 0 0"/>
   </joint>
